File: Hardware/Qwiic_BME688.brd (EAGLE design)
At the start: 25.4 x 25.4 mm, 45 parts, among them J2 QWIIC_RA, J4 QWIIC_RA, U1 BME688LGA

Commit message: Design review updates - buzzard labels
Parts:
- removed U$34: (no value), output:#3#3V#0
- removed U$4: (no value), output:#SCL#0
- added U$12: (no value), output:DEFAULT_ADR#_0X760
- added U$13: (no value), output:0X770
- added U$14: (no value), output:#3V3#0
- added U$16: (no value), output:#SDO#0
- added U$17, U$18: (no value), output:#CSB#0
- added U$19: (no value), output:#SDI#0
- added U$20: (no value), output:#SCK#0
- added U$8: (no value), output:#LED#0
- U$15: device SparkFun-Buzzard:I2C -> output:#3V3#0
- U$2: device output:#3#3V#0 -> output:#SDO#0
- U$3: device output:#SDA#0 -> output:#CSB#0
- U$6: device output:#PWR#0 -> output:#I2C#0
- U$9: device output:ADR#_0X760 -> output:0X760
- moved U$6 18.1 mm to (19.1, 18.5)
- moved U$15 17.4 mm to (14.0, 1.65), turned to 90 degrees
- moved U$3 15.1 mm to (13.2, 16.5), turned to 0 degrees
- moved U$9 14.0 mm to (17.5, 9.40), flipped to the bottom
- moved U$2 8.03 mm to (6.35, 1.65), flipped to the top
- moved U$11 4.12 mm to (13.6, 11.2)
- moved U$1 2.29 mm to (11.4, 1.65)
- moved U$33 2.29 mm to (11.4, 1.65)
- moved PWR 1.27 mm to (6.60, 7.62)
- moved D1 0.52 mm to (3.30, 6.86)
- moved R3 0.51 mm to (6.60, 6.86)
- moved ADR 0.51 mm to (11.4, 9.40)
- moved U$5 0.40 mm to (0.89, 8.13)
Routing:
- net 3.3V: track 56.2 -> 54.9 mm

Commit message: Engineering checklist
Parts:
- renumbered PWR to LED
Changed lines of the file:
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@@
 <?xml version="1.0" encoding="utf-8"?>
 <!DOCTYPE eagle SYSTEM "eagle.dtd">
-<eagle version="9.6.2">
+<eagle version="9.5.2">
 <drawing>
 <settings>
-<setting alwaysvectorfont="yes"/>
+<setting alwaysvectorfont="no"/>
 <setting keepoldvectorfont="yes"/>
 <setting verticaltext="up"/>
@@
 <layer number="37" name="tTest" color="7" fill="1" visible="no" active="yes"/>
 <layer number="38" name="bTest" color="7" fill="1" visible="no" active="yes"/>
-<layer number="39" name="tKeepout" color="4" fill="11" visible="no" active="yes"/>
+<layer number="39" name="tKeepout" color="4" fill="11" visible="yes" active="yes"/>
 <layer number="40" name="bKeepout" color="1" fill="11" visible="no" active="yes"/>
-<layer number="41" name="tRestrict" color="4" fill="10" visible="no" active="yes"/>
+<layer number="41" name="tRestrict" color="4" fill="10" visible="yes" active="yes"/>
 <layer number="42" name="bRestrict" color="1" fill="10" visible="no" active="yes"/>
 <layer number="43" name="vRestrict" color="2" fill="10" visible="no" active="yes"/>
@@
 <layer number="45" name="Holes" color="7" fill="1" visible="yes" active="yes"/>
 <layer number="46" name="Milling" color="3" fill="1" visible="no" active="yes"/>
-<layer number="47" name="Measures" color="7" fill="1" visible="no" active="yes"/>
+<layer number="47" name="Measures" color="7" fill="1" visible="yes" active="yes"/>
 <layer number="48" name="Document" color="7" fill="1" visible="no" active="yes"/>
 <layer number="49" name="Reference" color="7" fill="1" visible="no" active="yes"/>
@@
 HASL lead-free Finish</text>
 <dimension x1="5.08" y1="12.7" x2="5.08" y2="0" x3="-1.27" y3="6.35" textsize="1.778" textratio="15" layer="47" unit="inch"/>
-<dimension x1="8.89" y1="1.27" x2="0" y2="1.27" x3="4.445" y3="26.67" textsize="1.778" textratio="15" layer="47" unit="inch"/>
+<dimension x1="0" y1="0" x2="6.35" y2="0" x3="3.175" y3="26.67" textsize="1.778" textratio="15" layer="47" unit="inch"/>
 </plain>
 <attributes>
@@
 <attribute name="VALUE" value="2.2k" x="17.018" y="17.018" size="0.6096" layer="27" font="vector" ratio="20" rot="R90" align="top-center"/>
 </element>
-<element name="PWR" library="SparkFun-Jumpers" package="SMT-JUMPER_2_NC_TRACE_SILK" package3d_urn="urn:adsk.eagle:package:39281/1" value="JUMPER-SMT_2_NC_TRACE_SILK" x="6.604" y="7.62" smashed="yes" rot="MR0">
+<element name="LED" library="SparkFun-Jumpers" package="SMT-JUMPER_2_NC_TRACE_SILK" package3d_urn="urn:adsk.eagle:package:39281/1" value="JUMPER-SMT_2_NC_TRACE_SILK" x="6.604" y="7.62" smashed="yes" rot="MR0">
 <attribute name="NAME" x="6.604" y="8.763" size="0.6096" layer="26" font="vector" ratio="20" rot="MR0" align="bottom-center"/>
 </element>
@@
 <contactref element="J2" pad="2"/>
 <contactref element="J4" pad="2"/>
-<contactref element="PWR" pad="2"/>
+<contactref element="LED" pad="2"/>
 <contactref element="I2C" pad="2"/>
 <wire x1="20.328" y1="12.192" x2="20.32" y2="12.2" width="0.4064" layer="1"/>
@@
 <signal name="N$1">
 <contactref element="R3" pad="2"/>
-<contactref element="PWR" pad="1"/>
+<contactref element="LED" pad="1"/>
 <wire x1="8.509" y1="6.858" x2="7.454" y2="6.858" width="0.2032" layer="1"/>
 <via x="8.509" y="6.858" extent="1-16" drill="0.3048"/>
