File: Hardware/Qwiic_BME688.brd (EAGLE design)
At the start: 25.4 x 25.4 mm, 52 parts, among them J2 QWIIC_RA, J4 QWIIC_RA, U1 BME688LGA

Commit message: Rename PICO/POCI labels to SDO/SDI
Connections:
- net SDA/COPI renamed SDI/SDA
- net SDO/CIPO renamed SDO
Changed lines of the file:
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@@
 <wire x1="19.05" y1="2.54" x2="16.948" y2="4.642" width="0.2032" layer="1"/>
 </signal>
-<signal name="SDA/COPI">
+<signal name="SDI/SDA">
 <contactref element="J2" pad="3"/>
 <contactref element="J4" pad="3"/>
@@
 <wire x1="8.04" y1="9.232" x2="8.04" y2="10.16" width="0.2032" layer="1"/>
 </signal>
-<signal name="SDO/CIPO">
+<signal name="SDO">
 <contactref element="U1" pad="5"/>
 <contactref element="ADR" pad="2"/>
